File: hardware/kicad/acer-flow.kicad_pcb (KiCad board)
At the start: 2 copper layers, 0 parts

Commit message: Adding footprints. Starting layout
Parts:
- added C1: 0.1uF, Capacitor_SMD:C_0603_1608Metric, F.Cu at (121.5, 68.0)
- added C10: 22uF, Capacitor_SMD:C_0805_2012Metric, F.Cu at (189.6, 80.8)
- added C2: 100nF, Capacitor_SMD:C_0603_1608Metric, F.Cu at (145.5, 137.2)
- added C3: 1nF, Capacitor_SMD:C_0603_1608Metric, F.Cu at (194.0, 126.0)
- added C4: 1nF, Capacitor_SMD:C_0603_1608Metric, F.Cu at (195.2, 138.8)
- added C5: 10uF, Capacitor_SMD:C_0603_1608Metric, F.Cu at (44.5, 88.6)
- added C6: 10uF, Capacitor_SMD:C_0603_1608Metric, F.Cu at (191.5, 72.0)
- added C7: 10uF, Capacitor_SMD:C_0603_1608Metric, F.Cu at (164.5, 120.8)
- added C8: 10uF, Capacitor_SMD:C_0603_1608Metric, F.Cu at (172.5, 119.0)
- added C9: 22uF, Capacitor_SMD:C_0805_2012Metric, F.Cu at (189.6, 77.7)
- added D1: 1N5817, Diode_SMD:D_SOD-123, F.Cu at (62.5, 89.6)
- added D2: Blue 2.9V, LED_SMD:LED_0603_1608Metric, F.Cu at (67.4, 81.9)
- added D3: Green 3.2V, LED_SMD:LED_0603_1608Metric, F.Cu at (67.2, 85.6)
- added D4: LESD5D5.0CT1G, Diode_SMD:D_SOD-523, F.Cu at (192.8, 111.8)
- added D5: 1N5817, Diode_SMD:D_SOD-123, F.Cu at (167.2, 74.5)
- added J1: Conn_01x03, Connector_PinHeader_2.54mm:PinHeader_1x03_P2.54mm_Vertical, F.Cu at (205.0, 88.8)
- added J10: USB_B_Micro, Connector_USB:USB_Micro-B_Amphenol_10118194-0001LF_Horizontal, F.Cu at (203.9, 112.7)
- added J2: Conn_01x03, Connector_JST:JST_XH_B3B-XH-A_1x03_P2.50mm_Vertical, F.Cu at (141.2, 143.8)
- added J3: JTAG / SWD, Connector_PinHeader_1.27mm:PinHeader_2x05_P1.27mm_Vertical_SMD, F.Cu at (117.4, 106.3)
- added J4: Conn_01x04, Connector_JST:JST_XH_B4B-XH-A_1x04_P2.50mm_Vertical, F.Cu at (125.2, 144.0)
- added J5: Conn_01x01_Socket, Battery:BatteryClip_Keystone_54_D16-19mm, F.Cu at (73.2, 190.2)
- added J6: Conn_01x01_Socket, Battery:BatteryClip_Keystone_54_D16-19mm, F.Cu at (93.8, 190.4)
- added J7: Conn_01x01_Socket, Battery:BatteryClip_Keystone_54_D16-19mm, F.Cu at (74.0, 143.0)
- added J8: Conn_01x01_Socket, Battery:BatteryClip_Keystone_54_D16-19mm, F.Cu at (94.8, 143.0)
- added J9: Solar, Connector_JST:JST_XH_B2B-XH-A_1x02_P2.50mm_Vertical, F.Cu at (53.0, 78.1)
- added L1: 1uH, Inductor_SMD:L_Coilcraft_XAL4030-XXX, F.Cu at (183.8, 68.2)
- added Q1: AO3401A, Package_TO_SOT_SMD:SOT-23, F.Cu at (135.6, 128.8)
- added Q2: AO3401A, Package_TO_SOT_SMD:SOT-23, F.Cu at (166.6, 82.2)
- added R1: 4K7, Resistor_SMD:R_0603_1608Metric, F.Cu at (142.2, 137.2)
- added R2: 100, Resistor_SMD:R_0603_1608Metric, F.Cu at (129.8, 123.7)
- added R3: 100K, Resistor_SMD:R_0603_1608Metric, F.Cu at (129.8, 126.2)
- added R4: 180, Resistor_SMD:R_0603_1608Metric, F.Cu at (67.7, 96.1)
- added R5: 2k4, Resistor_SMD:R_0603_1608Metric, F.Cu at (65.2, 75.6)
- added R6: 100K, Resistor_SMD:R_0603_1608Metric, F.Cu at (157.9, 83.5)
- added R7: 100K, Resistor_SMD:R_0603_1608Metric, F.Cu at (174.4, 77.0)
- added R8: 732K, Resistor_SMD:R_0603_1608Metric, F.Cu at (182.7, 75.5)
- added R9: 100K, Resistor_SMD:R_0603_1608Metric, F.Cu at (180.4, 80.8)
- added SW1: RESET, Button_Switch_THT:SW_PUSH_6mm, F.Cu at (199.8, 126.0)
- added SW2: USER, Button_Switch_THT:SW_PUSH_6mm, F.Cu at (199.8, 136.2)
- added TP1: 5V, TestPoint:TestPoint_Pad_D1.5mm, F.Cu at (174.8, 85.5)
- added TP2: 3.3V, TestPoint:TestPoint_Pad_D1.5mm, F.Cu at (175.2, 108.0)
- added U1: WIO-SX1262, SB-Lib:Wio-SX1262-SB, F.Cu at (153.2, 61.2)
- added U2: 453-00001R, SB-Lib:45300001R, F.Cu at (124.0, 76.5)
- added U3: CN3158, Package_SO:SOIC-8-1EP_3.9x4.9mm_P1.27mm_EP2.41x3.3mm_ThermalVias, F.Cu at (55.8, 102.6)
- added U4: TLV75533PDBV, Package_TO_SOT_SMD:SOT-23-5, F.Cu at (166.8, 112.7)
- added U5: TPS61023, Package_TO_SOT_SMD:SOT-563, F.Cu at (174.5, 68.8)
